Commit message: Updates position of lidar sensor on car midway

File: aws-deepracer-controller-simple/simulation_ws/src/deepracer_simulation/urdf/racecar.xacro (robot description, xacro)
@@ -203,5 +203,5 @@
 <joint name="rplidar_joint" type="fixed">
     <axis xyz="0 1 0" />
-    <origin xyz="0.02 0 0.058" rpy="0 0 3.14"/>
+    <origin xyz="0.08 0 0.058" rpy="0 0 3.14"/>
     <parent link="base_link"/>
     <child link="laser"/>
